File: Hardware/beacon/beacon.kicad_pcb (KiCad board)
At the start: 2 copper layers, 13 x 27 mm, 32 parts, among them J1 Conn_01x05_Pin, J2 Conn_01x01_Pin, SW1 BOOT, U1 STM32WLE5CBUx, U2 XC6206P332MR, Y1 32MHz

Commit message: Files for version 1
Parts:
- added C15: 10u, Capacitor_SMD:C_0402_1005Metric, F.Cu at (106.4, 116.6)
- added H1: tooling, beacon_lib:toolinghole, F.Cu at (102.5, 100.4)
- added H2: tooling, beacon_lib:toolinghole, F.Cu at (113.0, 121.2)
- added L4: 15n, Inductor_SMD:L_0402_1005Metric, F.Cu at (107.5, 107.0)
- J1: value Conn_01x05_Pin -> DNP
- R1: value 0R -> DNP
- R2: value DNP -> 0R
Connections:
- R1 pad 1: /CONF_440 -> /CONF_220
- R2 pad 1: /CONF_868 -> /CONF_440
- U1 pad 1: /CONF_440 -> /CONF_220
- U1 pad 2: /CONF_868 -> /CONF_440
- U1 pad 20: unconnected-(U1-RFI_P-Pad20) -> /RFI_P
- U1 pad 21: unconnected-(U1-RFI_N-Pad21) -> /RFI_N
Routing:
- net /CONF_868: track 5.57 -> 0.00 mm
- net /CONF_220: track 0.00 -> 4.69 mm
- net /RFI_P: track 0.00 -> 3.97 mm
- net /RFI_N: track 0.00 -> 1.40 mm
- net GND: track 20.3 -> 21.1 mm, vias 32 -> 35
- net /CONF_440: track 4.69 -> 5.57 mm
Other:
- board text added: "Beacon"
- board text added: "JLCJLCJLCJLC"
- board text added: "V1.0"

Commit message: Audio testing
Parts:
- moved TP2 0.10 mm to (108.6, 118.9)
Other:
- board text added: "V1.1"
- board text added: "github.com/elvinc/rocketbeacon"
- board text removed: "V1.0"
Changed lines of the file:
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@@
   )
   (footprint "TestPoint:TestPoint_Pad_D1.0mm" (layer "F.Cu")
-    (at 108.6 119)
+    (at 108.6 118.9)
     (descr "SMD pad as test Point, diameter 1.0mm")
     (tags "test point SMD pad")
@@
     )
   )
-  (gr_rect (start 103.1 101.4) (end 112 106.9)
+  (gr_rect (start 103.5 101.4) (end 111 106.9)
     (stroke (width 0.15) (type solid)) (fill solid) (layer "B.SilkS"))
   (gr_line (start 110.7 120.35) (end 110.3 120.65)
@@
   (gr_circle (center 107.8 111.7) (end 122.8 111.7)
     (stroke (width 0.2) (type default)) (fill none) (layer "F.Fab"))
+  (gr_text "github.com/elvinc/rocketbeacon" (at 112.9 103.2 90) (layer "B.SilkS")
+    (effects (font (size 0.8 0.6) (thickness 0.15)) (justify left bottom mirror))
+  )
   (gr_text "JLCJLCJLCJLC" (at 110.6 119.4) (layer "B.SilkS")
     (effects (font (size 0.8 0.6) (thickness 0.15)) (justify left bottom mirror))
@@
     (effects (font (size 0.9 0.9) (thickness 0.15)) (justify left bottom))
   )
-  (gr_text "V1.0" (at 101.6 105) (layer "F.SilkS")
+  (gr_text "V1.1" (at 101.6 105) (layer "F.SilkS")
     (effects (font (size 0.8 0.8) (thickness 0.15)) (justify left bottom))
   )
