File: Hardware/beacon/beacon.kicad_pcb (KiCad board)
At the start: 2 copper layers, 13 x 27 mm, 36 parts, among them J1 DNP, J2 Conn_01x01_Pin, SW1 BOOT, U1 STM32WLE5CBUx, U2 XC6206P332MR, Y1 32MHz

Commit message: V1.1 beacon files
Parts:
- removed L4: 15n, Inductor_SMD:L_0402_1005Metric
- moved J1 0.08 mm to (112.5, 124.2)
Routing:
- net /RFI_P: track 3.97 -> 0.00 mm
- net /RFI_N: track 1.40 -> 0.00 mm
- net +3.3V: track 73.3 -> 74.3 mm, vias 5 -> 13
- added copper zone on F.Cu, net +3.3V
Other:
- board text added: "V1.1"
- board text added: "elvinc/rocketbeacon"
- board text removed: "V1.0"
