File: Hardware/beacon/beacon.kicad_sch (KiCad schematic)
At the start: 32 parts, among them J1 Conn_01x05_Pin, J2 Conn_01x01_Pin, SW1 BOOT, U1 STM32WLE5CBUx, U2 XC6206P332MR, Y1 32MHz

Commit message: Files for version 1
Parts:
- added C15: 10u, Capacitor_SMD:C_0402_1005Metric, symbol Device:C
- added H1, H2: tooling, beacon_lib:toolinghole, symbol Mechanical:MountingHole
- added L4: 15n, Inductor_SMD:L_0402_1005Metric, symbol Device:L
- J1: value Conn_01x05_Pin -> DNP
Connections:
- net +3.3V: now also C15.1
- net GND: now also C15.2
- net RFI_P: now reaches U1.20 (RFI_P)
- net RFI_P: now also L4.2
- net RFI_N: now reaches U1.21 (RFI_N)
- net RFI_N: now also L4.1
- no-connect marks 3 -> 24
Other:
- note added: "tooling holes"

Commit message: V1.1 beacon files
Parts:
- removed L4: 15n, Inductor_SMD:L_0402_1005Metric, symbol Device:L
- AE1, H1, H2, J1, J2, TP1, TP2: now left out of the parts list
Other:
- moved on the sheet: J2
